File: KiCad Files/esp32-detector.kicad_sch (KiCad schematic)
At the start: 89 parts, among them IC1 MC34119, J1 Coils Connector, J2 INTERFACE, U1 4066, U2 MCP602, U3 MCP602, U4 MCP602, U5 ESP32-WROOM-32, U6 LD1117S50TR, U7 LD1117S33TR

Commit message: Update sch and pcb files, Create .gitignore
Parts:
- C29, C33, C38, C39: footprint Capacitor_SMD:C_1206_3216Metric_Pad1.33x1.80mm_HandSolder -> Capacitor_SMD:C_1812_4532Metric_Pad1.57x3.40mm_HandSolder
- C32, C35: footprint Capacitor_SMD:C_1206_3216Metric_Pad1.33x1.80mm_HandSolder -> Capacitor_SMD:C_2220_5650Metric_Pad1.97x5.40mm_HandSolder
- L1: footprint Inductor_SMD:L_0805_2012Metric -> Inductor_SMD:L_1812_4532Metric_Pad1.30x3.40mm_HandSolder
Changed lines of the file:
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@@
       (effects (font (size 1.27 1.27)) (justify left))
     )
-    (property "Footprint" "Capacitor_SMD:C_1206_3216Metric_Pad1.33x1.80mm_HandSolder" (id 2) (at 54.61 149.86 0)
+    (property "Footprint" "Capacitor_SMD:C_1812_4532Metric_Pad1.57x3.40mm_HandSolder" (id 2) (at 54.61 149.86 0)
       (effects (font (size 1.27 1.27)) hide)
     )
@@
       (effects (font (size 1.27 1.27)) (justify left))
     )
-    (property "Footprint" "Capacitor_SMD:C_1206_3216Metric_Pad1.33x1.80mm_HandSolder" (id 2) (at 77.47 149.86 0)
+    (property "Footprint" "Capacitor_SMD:C_1812_4532Metric_Pad1.57x3.40mm_HandSolder" (id 2) (at 77.47 149.86 0)
       (effects (font (size 1.27 1.27)) hide)
     )
@@
       (effects (font (size 1.27 1.27)) (justify left))
     )
-    (property "Footprint" "Capacitor_SMD:C_1206_3216Metric_Pad1.33x1.80mm_HandSolder" (id 2) (at 54.61 120.65 0)
+    (property "Footprint" "Capacitor_SMD:C_2220_5650Metric_Pad1.97x5.40mm_HandSolder" (id 2) (at 54.61 120.65 0)
       (effects (font (size 1.27 1.27)) hide)
     )
@@
       (effects (font (size 1.27 1.27)) (justify left))
     )
-    (property "Footprint" "Capacitor_SMD:C_1206_3216Metric_Pad1.33x1.80mm_HandSolder" (id 2) (at 102.235 120.015 0)
+    (property "Footprint" "Capacitor_SMD:C_1812_4532Metric_Pad1.57x3.40mm_HandSolder" (id 2) (at 102.235 120.015 0)
       (effects (font (size 1.27 1.27)) hide)
     )
@@
     (property "Reference" "L1" (id 0) (at 59.055 139.065 90))
     (property "Value" "10mH" (id 1) (at 59.055 142.875 90))
-    (property "Footprint" "Inductor_SMD:L_0805_2012Metric" (id 2) (at 59.055 140.97 0)
+    (property "Footprint" "Inductor_SMD:L_1812_4532Metric_Pad1.30x3.40mm_HandSolder" (id 2) (at 59.055 140.97 0)
       (effects (font (size 1.27 1.27)) hide)
     )
@@
       (effects (font (size 1.27 1.27)) (justify left))
     )
-    (property "Footprint" "Capacitor_SMD:C_1206_3216Metric_Pad1.33x1.80mm_HandSolder" (id 2) (at 52.705 90.17 0)
+    (property "Footprint" "Capacitor_SMD:C_1812_4532Metric_Pad1.57x3.40mm_HandSolder" (id 2) (at 52.705 90.17 0)
       (effects (font (size 1.27 1.27)) hide)
     )
@@
       (effects (font (size 1.27 1.27)) (justify left))
     )
-    (property "Footprint" "Capacitor_SMD:C_1206_3216Metric_Pad1.33x1.80mm_HandSolder" (id 2) (at 29.21 116.84 0)
+    (property "Footprint" "Capacitor_SMD:C_2220_5650Metric_Pad1.97x5.40mm_HandSolder" (id 2) (at 29.21 116.84 0)
       (effects (font (size 1.27 1.27)) hide)
     )
@@
     )
     (path "/f481b64f-c3e7-4933-8efd-dd43c31cc7e1"
-      (reference "C29") (unit 1) (value "470u") (footprint "Capacitor_SMD:C_1206_3216Metric_Pad1.33x1.80mm_HandSolder")
+      (reference "C29") (unit 1) (value "470u") (footprint "Capacitor_SMD:C_1812_4532Metric_Pad1.57x3.40mm_HandSolder")
     )
     (path "/f1f99eba-0018-4b99-b8f5-9a8c24b5c8bf"
@@
     )
     (path "/f9a6ac91-d68c-456b-8585-94b3d8e86987"
-      (reference "C32") (unit 1) (value "100u") (footprint "Capacitor_SMD:C_1206_3216Metric_Pad1.33x1.80mm_HandSolder")
+      (reference "C32") (unit 1) (value "100u") (footprint "Capacitor_SMD:C_2220_5650Metric_Pad1.97x5.40mm_HandSolder")
     )
     (path "/7e3ed924-7bd4-439e-9b38-53a4bf12619d"
-      (reference "C33") (unit 1) (value "470u") (footprint "Capacitor_SMD:C_1206_3216Metric_Pad1.33x1.80mm_HandSolder")
+      (reference "C33") (unit 1) (value "470u") (footprint "Capacitor_SMD:C_1812_4532Metric_Pad1.57x3.40mm_HandSolder")
     )
     (path "/55dd072f-ba8c-4b26-9c3a-4018b66d821e"
@@
     )
     (path "/6c484191-d3e1-48ff-af2e-f0d7d9278f03"
-      (reference "C35") (unit 1) (value "470u") (footprint "Capacitor_SMD:C_1206_3216Metric_Pad1.33x1.80mm_HandSolder")
+      (reference "C35") (unit 1) (value "470u") (footprint "Capacitor_SMD:C_2220_5650Metric_Pad1.97x5.40mm_HandSolder")
     )
     (path "/6dc60ca2-559c-4934-9b56-3feb6de94aa4"
@@
     )
     (path "/044fa026-f2ba-4022-8462-55805448e937"
-      (reference "C38") (unit 1) (value "470u") (footprint "Capacitor_SMD:C_1206_3216Metric_Pad1.33x1.80mm_HandSolder")
+      (reference "C38") (unit 1) (value "470u") (footprint "Capacitor_SMD:C_1812_4532Metric_Pad1.57x3.40mm_HandSolder")
     )
     (path "/2997039c-af2f-4a49-9e71-a563e0816db6"
-      (reference "C39") (unit 1) (value "470u") (footprint "Capacitor_SMD:C_1206_3216Metric_Pad1.33x1.80mm_HandSolder")
+      (reference "C39") (unit 1) (value "470u") (footprint "Capacitor_SMD:C_1812_4532Metric_Pad1.57x3.40mm_HandSolder")
     )
     (path "/09b320e3-e745-41af-8e20-4b0fd4efe3bc"
@@
     )
     (path "/e77775c5-552f-49b3-900f-a86912e85311"
-      (reference "L1") (unit 1) (value "10mH") (footprint "Inductor_SMD:L_0805_2012Metric")
+      (reference "L1") (unit 1) (value "10mH") (footprint "Inductor_SMD:L_1812_4532Metric_Pad1.30x3.40mm_HandSolder")
     )
     (path "/a7092e7b-f87a-4f5a-ba8e-c3f8d915f6af"
